File: 01-Hardware/Fuente_Simetrica/Fuente_Simetrica.kicad_pcb (KiCad board)
At the start: 2 copper layers, 107 x 64.5 mm, 24 parts, among them J1 AC_IN, J2 VCC_CONN, U1 L7812, U2 L7912

Commit message: Últimos cambios PCB
Parts:
- C3, C4, C5, C6: footprint Capacitor_THT:C_Disc_D5.0mm_W2.5mm_P2.50mm -> Capacitor_THT:C_Disc_D5.0mm_W2.5mm_P5.00mm
- moved C5 1.03 mm to (160.0, 130.0)
- moved C4 1.00 mm to (152.5, 132.8)
Routing:
- net Net-(D1-A): track 53.6 -> 49.4 mm
- net Net-(J2-Pin_1): track 29.3 -> 32.5 mm
- net GND: track 198.1 -> 197.1 mm
- net Net-(J2-Pin_3): track 26.2 -> 25.7 mm

Commit message: Últimos cambios PCB
Routing:
- net GND: track 197.1 -> 195.2 mm
Changed lines of the file:
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@@
+	)
+	(segment
+		(start 128.5 129)
+		(end 130.75 131.25)
+		(width 1.5)
+		(layer "B.Cu")
+		(net 2)
 	)
 	(segment
@@
 	)
 	(segment
-		(start 137.5 133.5)
-		(end 142 129)
-		(width 1.5)
-		(layer "B.Cu")
-		(net 2)
-	)
-	(segment
 		(start 171 123)
 		(end 166.5 127.5)
@@
 	)
 	(segment
+		(start 142 129)
+		(end 139.75 131.25)
+		(width 1.5)
+		(layer "B.Cu")
+		(net 2)
+	)
+	(segment
 		(start 115.5 118.5)
 		(end 109 125)
@@
 	)
 	(segment
-		(start 133 133.5)
-		(end 133.692994 133.5)
-		(width 1.2)
+		(start 139.75 131.25)
+		(end 130.75 131.25)
+		(width 1.5)
 		(layer "B.Cu")
 		(net 2)
@@
 		(start 142.487246 119)
 		(end 142 119.487246)
-		(width 1.5)
-		(layer "B.Cu")
-		(net 2)
-	)
-	(segment
-		(start 133.692994 133.5)
-		(end 137.5 133.5)
 		(width 1.5)
 		(layer "B.Cu")
@@
 	)
 	(segment
-		(start 128.5 129)
-		(end 133 133.5)
-		(width 1.2)
-		(layer "B.Cu")
-		(net 2)
-	)
-	(segment
 		(start 167.04 141)
 		(end 161.54 135.5)
@@
 	)
 	(segment
-		(start 133.5 136.5)
-		(end 133.3 136.3)
-		(width 1.2)
-		(layer "B.Cu")
-		(net 3)
-	)
-	(segment
-		(start 133.3 136.3)
-		(end 133.3 136.127308)
+		(start 140.28 134.78)
+		(end 142 136.5)
 		(width 1.2)
 		(layer "B.Cu")
@@
 	)
 	(segment
-		(start 142 136.5)
-		(end 134.5 136.5)
-		(width 1.5)
-		(layer "B.Cu")
-		(net 3)
-	)
-	(segment
-		(start 134.5 136.5)
-		(end 133.5 136.5)
-		(width 1.2)
-		(layer "B.Cu")
-		(net 3)
-	)
-	(segment
-		(start 131.952692 134.78)
-		(end 131.78 134.78)
-		(width 1.2)
-		(layer "B.Cu")
-		(net 3)
-	)
-	(segment
 		(start 159 138.5)
 		(end 159 135.5)
@@
 	)
 	(segment
-		(start 133.3 136.127308)
-		(end 131.952692 134.78)
+		(start 131.78 134.78)
+		(end 140.28 134.78)
 		(width 1.2)
 		(layer "B.Cu")
@@
 		(start 172.5 103.5)
 		(end 172.5 105.5)
-		(width 1.2)
+		(width 1.5)
 		(layer "B.Cu")
 		(net 5)
